File: projects/pitechoid/video/video_v1.kicad_pcb (KiCad board)
At the start: 2 copper layers, 99.1 x 99.1 mm, 60 parts, among them CN1 HEADER_2x16_p2.54_TH_RA, CN1 RCA_DUAL_RS212, CN2 SUB-D15, CN3 2x8_RA_Fem, CN3 HEADER_2x8_p2.54_TH_RA, U1 TVP5150AM1T, U3 LM1117-ADJ, U4 ADV7123, X1 14.31818MHz

Commit message: update
Parts:
- removed the CN1 at (97.8, 125.7)
- removed the CN2 at (174.3, 142.2)
- removed the CN3 at (97.8, 72.4)
- removed the X1 at (123.6, 85.1)
- added CN4: RCA_DUAL_RS212, Footprints:RCA_DUAL_RS212, F.Cu at (131.9, 62.3)
- added CN5: HEADER_2x8_p2.54_TH_RA, Footprints:HEADER_2x8_M_p2.54_TH_RA, F.Cu at (135.4, 72.0)
- C13: value xxnF -> 100nF
- CN1: value RCA_DUAL_RS212 -> HEADER_2x16_p2.54_TH_RA; footprint Footprints:RCA_DUAL_RS212 -> Footprints:HEADER_2x16_M_p2.54_TH_RA
- CN3: value 2x8_RA_Fem -> HEADER_2x8_p2.54_TH_RA; footprint headers_eag:2X08_90 -> Footprints:HEADER_2x8_M_p2.54_TH_RA
- R12: value 1K -> 10K
- R14: value 2K2 -> 50R
- moved CN1 64.8 mm to (103.3, 120.7), turned to 90 degrees
- moved CN3 52.0 mm to (102.6, 73.7)
- moved X1 4.45 mm to (147.3, 136.5)
- moved C10 3.32 mm to (135.4, 138.4)
- moved C9 1.95 mm to (135.0, 134.6)
- moved C5 0.78 mm to (134.3, 127.0)
- moved R16 0.78 mm to (129.9, 88.1)
- moved C1 0.06 mm to (131.2, 67.3)
- moved C11 0.06 mm to (123.6, 88.9)
- moved C13 0.06 mm to (130.5, 127.6)
- moved C2 0.06 mm to (192.6, 105.3)
- moved C2 0.06 mm to (133.7, 67.3)
- moved C3 0.06 mm to (192.6, 108.1)
- moved C3 0.06 mm to (126.1, 72.4)
- moved C4 0.06 mm to (132.5, 72.4)
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Connections:
- net Net-(C10-Pad2) renamed /IN1_CN
- net Net-(C9-Pad2) renamed /IN2_CN
- C13 pad 1: unconnected-(C11-Pad1) -> +3V3
- C13 pad 2: unconnected-(C11-Pad2) -> GND
- CN1 pad 3: N$7 -> /VGA_VSYNC
- CN1 pad 4: N$8 -> unconnected-(CN1-Pad4)
- CN2 pad H1: (no net) -> GND
- CN2 pad H2: (no net) -> GND
- CN3 pad 10: +5V -> /+5V
- CN3 pad 11: +5V -> /+5V
- CN3 pad 12: +5V -> /+5V
- CN3 pad 13: +12V -> /+12V
- CN3 pad 14: +12V -> /+12V
- CN3 pad 15: +12V -> /+12V
- CN3 pad 16: +12V -> /+12V
- CN3 pad 9: +5V -> /+5V
- R12 pad 1: N$6 -> /TVP_RSTn
- R12 pad 2: +1V8 -> +3V3
- R14 pad 1: GND -> /VGA_VSYNC
- R14 pad 2: N$6 -> Net-(CN2-Pad14)
Routing:
- net +3V3: track 31.4 -> 0.20 mm
- net +1V8: track 29.5 -> 0.00 mm
- net N$17: track 24.0 -> 0.00 mm
- net N$18: track 18.5 -> 0.00 mm
- net OUT_R: track 14.0 -> 0.00 mm
- net OUT_G: track 10.5 -> 0.00 mm
- net N$7: track 10.0 -> 0.00 mm
- net OUT_B: track 7.89 -> 0.00 mm
- net N$9: track 4.80 -> 0.00 mm
