File: projects/pitechoid/video/video_v1.kicad_sch (KiCad schematic)
At the start: 38 parts, among them CN1 HEADER_2x16_p2.54_TH_RA, CN2 SUB-D15, CN3 HEADER_2x8_p2.54_TH_RA, U1 TVP5150AM1T, U3 LM1117-ADJ, U4 ADV7123, X1 14.31818MHz

Commit message: update
Parts:
- added CN4: RCA_DUAL_RS212, Footprints:RCA_DUAL_RS212, symbol connectors:RCA_DUAL_RS212
- added CN5: HEADER_2x8_p2.54_TH_RA, Footprints:HEADER_2x8_M_p2.54_TH_RA, symbol headers:HEADER_2X8
- added R21, R22: 10K, Footprints:R1206, symbol passives:Resistor
- CN1: footprint Footprints:HEADER_2x16_p2.54_TH_RA -> Footprints:HEADER_2x16_M_p2.54_TH_RA
- CN3: footprint Footprints:HEADER_2x8_p2.54_TH_RA -> Footprints:HEADER_2x8_M_p2.54_TH_RA
Connections:
- net CLK4 is gone; now on net VGA_G4: CN1.11
- net CLK5 is gone; now on net VGA_G7: CN1.10
- net CLK6 is gone; now on net VGA_G6: CN1.9
- net CVBS_RSTN is gone; now on net TVP_RSTn: CN1.29
- net VGA_B3 is gone; now on net GND: U4.19 (B5)
- net VGA_G2 is gone; now on net GND: U4.5 (G4)
- net VGA_G3 is gone; now on net GND: U4.6 (G5)
- net VGA_R2 is gone; now on net GND: U4.43 (R4)
- net VGA_R3 is gone; now on net GND: U4.44 (R5)
- net +12V: now also CN5.13, CN5.14, CN5.15, CN5.16
- net +3V3: now also CN5.5, CN5.6, CN5.7, CN5.8, R21.2, R22.2
- net +5V: now also CN5.10, CN5.11, CN5.12, CN5.9
- net CVBS_CLK: now also CN1.31; no longer CN1.30
- net GND: now also CN2.H1 (1), CN2.H2 (1), U4.18 (B4), CN4.1 (GND1), CN4.2 (GND2), CN5.1, CN5.2, CN5.3, CN5.4
- net SCL: now also R21.1
- net SDA: now also CN1.30, R22.1; no longer CN1.31
- net VGA_B5: now also CN1.6
- net VGA_B6: now also CN1.19
- net VGA_B7: now also CN1.17
- net VGA_CLOCK: now also CN1.18
- net VGA_G5: now also CN1.12
- net VGA_HSYNC: now also CN1.4
- net VGA_R4: now also CN1.15
- net VGA_R5: now also CN1.16
- net VGA_R6: now also CN1.13
- net VGA_R7: now also CN1.14
- net VGA_~{BLANK}: now also CN1.7
- net VGA_~{SYNC}: now also CN1.8
- net IN1_CN: now reaches C10.2, R19.2
- net IN1_CN: now also CN4.3 (IN1)
- net IN2_CN: now reaches C9.2, R20.2
- net IN2_CN: now also CN4.4 (IN2)
- removed net VGA_B2: CN1.7, U4.18 (B4)
Other:
- note added: "3.3V to 1.8V"
- moved on the sheet: C1, C10, C13, C14, C15, C16, C17, C18, C2, C3, C5, C6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
